Commit message: urdf modification

File: mecanumbot_description/urdf/mecanumbot.urdf (robot description, URDF)
Before this commit: robot mecanumbot, 6 links, 5 joints
Links:
- added link imu_link, mass ${imu_mass}; collision box size=${imu_size_x} ${imu_size_y} ${imu_size_z}; visual box size=${imu_size_x} ${imu_size_y} ${imu_size_z}
- added link laser_frame, mass ${lidar_mass}; collision cylinder length=${lidar_width} radius=${lidar_radius}; visual cylinder length=${lidar_width} radius=${lidar_radius}
Joints:
- added joint imu_joint: type fixed, parent base_link, child imu_link, origin xyz=${imu_offset_x} ${imu_offset_y} ${imu_offset_z} rpy=0 0 0
- added joint laser_joint: type fixed, parent base_link, child laser_frame, origin xyz=${-lidar_offset_x} ${-lidar_offset_y} ${lidar_offset_z} rpy=0 0 0
